File: Apple1Cartridge.kicad_pcb (KiCad board)
At the start: 2 copper layers, 110.1 x 77.7 mm, 16 parts

Commit message: Fixed element values on schematics
Parts:
- BANK1: footprint Package_DIP:DIP-14_W7.62mm_Socket_LongPads -> Package_DIP:DIP-14_W7.62mm_LongPads
- DECODER1: footprint Package_DIP:DIP-24_W7.62mm_Socket_LongPads -> Package_DIP:DIP-24_W7.62mm_LongPads
- MODE_SWITCH1: renamed from MODE_SWITCH; value SW_SPDT -> MODE_SWITCH
- RAM1, ROM1: footprint Package_DIP:DIP-28_W15.24mm_Socket_LongPads -> Package_DIP:DIP-28_W15.24mm_LongPads
- RAM2: footprint Package_DIP:DIP-28_W15.24mm_Socket -> Package_DIP:DIP-28_W15.24mm
